Commit message: 函数版 Thymio 小机器人添加碰撞体积+质量,惯性属性，添加 Gazebo.xacro 属性文件

File: src/thymio_description/urdf/example/example.urdf.xacro (robot description, xacro)
@@ -3,4 +3,5 @@
     <!-- 依赖库，类似 c++ 头文件或者 python import -->
     <xacro:include filename="example_materials.xacro"/>
+    <xacro:include filename="example_inertia.xacro"/>
     <!-- 定义变量 -->
     <xacro:property name="base_link_length" value="0.2"/>
@@ -9,4 +10,6 @@
     <xacro:property name="second_link_length" value="0.8"/>
     <xacro:property name="second_link_radius" value="0.05"/>
+    <xacro:property name="base_link_mass" value="0.5"/>   <!-- Mass in [kg] -->
+    <xacro:property name="second_link_mass" value="0.2"/> <!-- Mass in [kg] -->
     <!-- 自定义函数 -->
     <xacro:macro name="box" params="length width height">
@@ -22,4 +25,12 @@
             <material name="green"/>
         </visual>
+        <collision>
+            <origin xyz="0 0 ${base_link_height / 2.0}"  rpy="0 0 0"/>
+            <geometry>
+                <xacro:box length="${base_link_length}" width="${base_link_width}" height="${base_link_height}"/>
+            </geometry>
+        </collision>
+        <xacro:box_inertia m="${base_link_mass}" l="${base_link_length}" w="${base_link_width}" h="${base_link_height}"
+                        xyz="0 0 ${base_link_height / 2.0}"  rpy="0 0 0"/>
     </link>
     <link name="second_link">
@@ -31,4 +42,12 @@
             <material name="blue"/>
         </visual>
+        <collision>
+            <origin xyz="${second_link_length / 2.0} 0 0" rpy="0 ${pi / 2.0} 0"/>
+            <geometry>
+                <cylinder length="${second_link_length}" radius="${second_link_radius}"/>
+            </geometry>
+        </collision>
+        <xacro:cylinder_inertia m="${second_link_mass}" r="${second_link_radius}" h="${second_link_length}"
+                                xyz="${second_link_length / 2.0} 0 0" rpy="0 ${pi / 2.0} 0"/>
     </link>
     <joint name="second_link_joint" type="fixed">

File: src/thymio_description/urdf/thymio/thymio.urdf.xacro (robot description, xacro)
@@ -4,29 +4,27 @@
     <xacro:include filename="materials.xacro"/>
     <xacro:include filename="thymio_chassis.xacro"/>
+    <xacro:include filename="gazebo.xacro"/>
     <!-- 建模 -->
     <!-- 创建 基座 -->
     <link name="base_link">
-        <visual>
-            <origin xyz="0 0 ${base_link_height/2 + ground_offset}"  rpy="0 0 0"/>
-            <geometry>
-                <xacro:box length="${base_link_length}"
-                           width="${base_link_width}"
-                           height="${base_link_height}"/>
-            </geometry>
-            <material name="white"/>
-        </visual>
+        <xacro:build_base length="${base_link_length}"
+                          width="${base_link_width}"
+                          height="${base_link_height}"
+                          mass="${base_mass}" />
     </link>
     <!-- 创建 轮子1-->
     <link name="wheel_1">
       <xacro:build_wheel length="${wheel_link_length}"
-                         radius="${wheel_link_radius}"/>
+                         radius="${wheel_link_radius}"
+                         mass="${wheel_mass}"/>
     </link>
     <!-- 创建 轮子2-->
     <link name="wheel_2">
       <xacro:build_wheel length="${wheel_link_length}"
-                         radius="${wheel_link_radius}"/>
+                         radius="${wheel_link_radius}"
+                         mass="${wheel_mass}"/>
     </link>
     <!-- 创建 万向轮-->
-    <link name="caster_wheel">
+    <link name="caster_wheel_link">
         <visual>
             <origin xyz="0 0 0" rpy="0 0 0"/>
@@ -36,4 +34,10 @@
             <material name="white"/>
         </visual>
+        <collision>
+            <origin xyz="0 0 0" rpy="0 0 0"/>
+            <geometry>
+                <sphere radius="${caster_wheel_ball_radius}"/>
+            </geometry>
+        </collision>
     </link>
     <!-- 关节 -->
@@ -43,4 +47,5 @@
         <origin xyz="${front_axis} 0.05 ${wheel_link_radius}" rpy="0 0 0"/>
         <axis xyz="0 1 0"/>
+        <dynamics damping="0.1" friction="0.2"/>   <!-- 添加阻尼，摩擦-->
     </joint>
     <joint name="wheel_2_joint" type="continuous">
@@ -49,10 +54,12 @@
         <origin xyz="${front_axis} -0.05 ${wheel_link_radius}" rpy="0 0 0"/>
         <axis xyz="0 1 0"/>
+        <dynamics damping="0.1" friction="0.2"/>
     </joint>
     <joint name="caster_wheel_joint" type="continuous">
         <parent link="base_link"/>
-        <child link="caster_wheel"/>
+        <child link="caster_wheel_link"/>
         <origin xyz="${rear_axis} 0.0 ${caster_wheel_ball_radius}" rpy="0 0 0"/>
         <axis xyz="0 1 0"/>
+        <dynamics damping="0.1" friction="0.2"/>
     </joint>
 </robot>

File: src/thymio_description/urdf/thymio/thymio_chassis.xacro (robot description, xacro)
@@ -1,8 +1,12 @@
 <?xml version="1.0"?>
 <robot xmlns:xacro="http://www.ros.org/wiki/xacro">
-    <!-- 机器人底盘参数 -->
-    <!-- 定义变量 -->
+  <!-- 机器人底盘参数 -->
+  <!-- 定义变量 -->
+    <!-- 定义基本单位 -->
     <xacro:property name="mm" value="0.001"/>
     <xacro:property name="cm" value="0.01"/>
+    <xacro:property name="g"  value="0.001"/>
+    <xacro:property name="kg" value="1.0"/>
+    <!-- 定义尺寸 -->
     <xacro:property name="ground_offset"     value="${4.5*mm}"/>
     <xacro:property name="base_link_length"  value="${11*cm}"/>
@@ -13,6 +17,12 @@
     <xacro:property name="caster_wheel_ball_radius" value="${9*mm}"/>
     <xacro:property name="front_axis" value="${2.5*cm}"/>
-    <xacro:property name="rear_axis" value="${-3.5*cm}"/>
-    <!-- 自定义函数 1级 -->
+    <xacro:property name="rear_axis"  value="${-3.5*cm}"/>
+    <!-- 定义重量 -->
+    <xacro:property name="mass"              value="${270*g}"/>
+    <xacro:property name="base_mass"         value="${mass*0.8*0.95}"/>
+    <xacro:property name="wheel_mass"        value="${mass*0.2 / 2}"/>
+    <xacro:property name="caster_wheel_mass" value="${mass*0.8*0.05}"/>
+  <!-- 自定义函数 1级 -->
+    <!-- 定义几何图形函数 -->
     <xacro:macro name="box" params="length width height">
         <box size="${length} ${width} ${height}"/>
@@ -24,6 +34,59 @@
         <sphere radius="${radius}"/>
     </xacro:macro>
+    <!-- 定义转动惯量函数 -->
+    <xacro:macro name="box_inertia" params="m l w h xyz rpy">
+    <inertial>
+        <origin xyz="${xyz}" rpy="${rpy}"/>
+        <mass value="${m}"/>
+        <inertia
+        ixx="${(m/12) * (w*w + h*h)}"
+        ixy="0" ixz="0"
+        iyy="${(m/12) * (l*l + h*h)}"
+        iyz="0"
+        izz="${(m/12) * (l*l + w*w)}"/>
+    </inertial>
+    </xacro:macro>
+    <xacro:macro name="cylinder_inertia" params="m r h xyz rpy">
+        <inertial>
+            <origin xyz="${xyz}" rpy="${rpy}"/>
+            <mass value="${m}" />
+            <inertia ixx="${(m/12) * (3*r*r + h*h)}" ixy="0" ixz="0"
+                    iyy="${(m/12) * (3*r*r + h*h)}" iyz="0"
+                    izz="${(m/2) * (r*r)}"/>
+        </inertial>
+    </xacro:macro>
     <!-- 自定义函数 2级 -->
-    <xacro:macro name="build_wheel" params="length radius">
+    <!-- 创建主体 -->
+    <xacro:macro name="build_base" params="length width height mass">
+        <!-- 视觉形状+颜色 -->
+        <visual>
+            <origin xyz="0 0 ${base_link_height/2 + ground_offset}"  rpy="0 0 0"/>
+            <geometry>
+                <xacro:box length="${length}"
+                           width="${width}"
+                           height="${height}"/>
+            </geometry>
+            <material name="white"/>
+        </visual>
+        <!-- 碰撞体积 -->
+        <collision>
+            <origin xyz="0 0 ${base_link_height/2 + ground_offset}"  rpy="0 0 0"/>
+            <geometry>
+                <xacro:box length="${length}"
+                           width="${width}"
+                           height="${height}"/>
+            </geometry>
+        </collision>
+        <!-- 惯性 -->
+        <xacro:box_inertia m="${mass}"
+                           l="${length}"
+                           w="${width}"
+                           h="${height}"
+                           xyz="0 0 ${base_link_height/2 + ground_offset}"
+                           rpy="0 0 0" />
+    </xacro:macro>
+    <!-- 创建轮子 -->
+    <xacro:macro name="build_wheel" params="length radius mass">
+        <!-- 视觉形状+颜色 -->
         <visual>
             <origin xyz="0 0 0" rpy="${pi/2.0} 0 0"/>
@@ -33,4 +96,19 @@
             </geometry>
             <material name="black"/>
-        </visual>     </xacro:macro>
+        </visual>
+        <!-- 碰撞体积 -->
+        <collision>
+            <origin xyz="0 0 0" rpy="${pi/2.0} 0 0"/>
+            <geometry>
+                <xacro:wheel length="${length}"
+                             radius="${radius}"/>
+            </geometry>
+        </collision>
+        <!-- 惯性 -->
+        <xacro:cylinder_inertia m="${mass}"
+                                r="${radius}"
+                                h="${length}"
+                                xyz="0 0 0"
+                                rpy="${pi/2.0} 0 0" />
+     </xacro:macro>
 </robot>
