Commit message: 添加传感器版本

File: src/thymio_description/urdf/thymio/thymio.urdf.xacro (robot description, xacro)
@@ -5,4 +5,5 @@
     <xacro:include filename="thymio_chassis.xacro"/>
     <xacro:include filename="gazebo.xacro"/>
+    <xacro:include filename="proximity_sensors.xacro"/>
     <!-- 建模 -->
     <!-- 创建 基座 -->

File: src/thymio_description/urdf/thymio/thymio_chassis.xacro (robot description, xacro)
@@ -10,5 +10,5 @@
     <!-- 定义尺寸 -->
     <xacro:property name="ground_offset"     value="${4.5*mm}"/>
-    <xacro:property name="base_link_length"  value="${11*cm}"/>
+    <xacro:property name="base_link_length"  value="${9.1*cm}"/>
     <xacro:property name="base_link_width"   value="${11.2*cm}"/>
     <xacro:property name="base_link_height"  value="${4.4*cm}"/>
